File: PCB_Design/picoAWG.kicad_pcb (KiCad board)
At the start: 4 copper layers, 0 parts

Commit message: KiCAD file update, completed PCB
Parts:
- added C1: 27p, Capacitor_SMD:C_0603_1608Metric, F.Cu at (88.3, 102.9)
- added C10: 0.1u, Capacitor_SMD:C_0603_1608Metric, F.Cu at (76.0, 102.9)
- added C100: 0.1u, Capacitor_SMD:C_0603_1608Metric, F.Cu at (162.2, 64.2)
- added C101: 0.1u, Capacitor_SMD:C_0603_1608Metric, F.Cu at (157.2, 68.0)
- added C102: 0.1u, Capacitor_SMD:C_0603_1608Metric, F.Cu at (161.7, 79.4)
- added C103: 0.1u, Capacitor_SMD:C_0603_1608Metric, F.Cu at (156.9, 83.7)
- added C104: 1u, Capacitor_SMD:C_0603_1608Metric, F.Cu at (177.1, 86.1)
- added C105: 1u, Capacitor_SMD:C_0603_1608Metric, F.Cu at (177.1, 82.9)
- added C106: 1u, Capacitor_SMD:C_0603_1608Metric, F.Cu at (177.0, 70.3)
- added C107: 1u, Capacitor_SMD:C_0603_1608Metric, F.Cu at (177.0, 67.2)
- added C108: 0.1u, Capacitor_SMD:C_0603_1608Metric, F.Cu at (124.2, 45.2)
- added C109: 0.1u, Capacitor_SMD:C_0603_1608Metric, F.Cu at (140.2, 43.5)
- added C11: 0.1u, Capacitor_SMD:C_0603_1608Metric, F.Cu at (71.5, 101.9)
- added C110: 0.1u, Capacitor_SMD:C_0603_1608Metric, F.Cu at (140.2, 45.4)
- added C111: 1.5p, Capacitor_SMD:C_0603_1608Metric, F.Cu at (149.5, 51.8)
- added C112: 1.5p, Capacitor_SMD:C_0603_1608Metric, F.Cu at (149.5, 54.9)
- added C113: 1.5p, Capacitor_SMD:C_0603_1608Metric, F.Cu at (149.5, 36.5)
- added C114: 1.5p, Capacitor_SMD:C_0603_1608Metric, F.Cu at (149.5, 33.5)
- added C115: 0.1u, Capacitor_SMD:C_0603_1608Metric, F.Cu at (125.9, 41.9)
- added C116: 0.1u, Capacitor_SMD:C_0603_1608Metric, F.Cu at (136.7, 44.5)
- added C117: 0.1u, Capacitor_SMD:C_0603_1608Metric, F.Cu at (127.3, 46.2)
- added C118: 0.1u, Capacitor_SMD:C_0603_1608Metric, F.Cu at (132.4, 38.5)
- added C119: 0.1u, Capacitor_SMD:C_0603_1608Metric, F.Cu at (132.4, 49.8)
- added C12: 0.1u, Capacitor_SMD:C_0603_1608Metric, F.Cu at (72.4, 89.8)
- added C120: 1.5p, Capacitor_SMD:C_0603_1608Metric, F.Cu at (149.5, 45.7)
- added C121: 1.5p, Capacitor_SMD:C_0603_1608Metric, F.Cu at (149.5, 48.7)
- added C122: 1.5p, Capacitor_SMD:C_0603_1608Metric, F.Cu at (149.5, 39.6)
- added C123: 1.5p, Capacitor_SMD:C_0603_1608Metric, F.Cu at (149.5, 42.6)
- added C124: 0.1u, Capacitor_SMD:C_0603_1608Metric, F.Cu at (164.2, 40.7)
- added C125: 0.1u, Capacitor_SMD:C_0603_1608Metric, F.Cu at (167.5, 36.8)
- added C126: 0.1u, Capacitor_SMD:C_0603_1608Metric, F.Cu at (163.8, 56.9)
- added C127: 0.1u, Capacitor_SMD:C_0603_1608Metric, F.Cu at (169.1, 52.8)
- added C128: 0.1u, Capacitor_SMD:C_0603_1608Metric, F.Cu at (162.3, 32.2)
- added C129: 0.1u, Capacitor_SMD:C_0603_1608Metric, F.Cu at (157.3, 36.1)
- added C13: 0.1u, Capacitor_SMD:C_0603_1608Metric, F.Cu at (60.0, 95.4)
- added C130: 0.1u, Capacitor_SMD:C_0603_1608Metric, F.Cu at (161.8, 47.5)
- added C131: 0.1u, Capacitor_SMD:C_0603_1608Metric, F.Cu at (157.0, 51.8)
- added C132: 1u, Capacitor_SMD:C_0603_1608Metric, F.Cu at (177.2, 54.1)
- added C133: 1u, Capacitor_SMD:C_0603_1608Metric, F.Cu at (177.2, 51.0)
- added C134: 1u, Capacitor_SMD:C_0603_1608Metric, F.Cu at (177.1, 38.4)
- added C135: 1u, Capacitor_SMD:C_0603_1608Metric, F.Cu at (177.1, 35.3)
- added C136: 1n, Capacitor_SMD:C_0603_1608Metric, F.Cu at (217.7, 60.0)
- added C137: 1n, Capacitor_SMD:C_0603_1608Metric, F.Cu at (225.7, 60.0)
- added C138: 0.1u, Capacitor_SMD:C_0603_1608Metric, F.Cu at (246.8, 63.5)
- added C139: 0.1u, Capacitor_SMD:C_0603_1608Metric, F.Cu at (215.8, 51.5)
- added C14: 0.1u, Capacitor_SMD:C_0603_1608Metric, F.Cu at (68.0, 94.7)
- added C140: 0.1u, Capacitor_SMD:C_0603_1608Metric, F.Cu at (220.0, 56.7)
- added C141: 0.1u, Capacitor_SMD:C_0603_1608Metric, F.Cu at (223.9, 51.5)
- added C142: 0.1u, Capacitor_SMD:C_0603_1608Metric, F.Cu at (228.0, 56.7)
- added C143: 0.1u, Capacitor_SMD:C_0603_1608Metric, F.Cu at (224.8, 47.6)
- added C144: 0.1u, Capacitor_SMD:C_0603_1608Metric, F.Cu at (220.8, 47.6)
- added C145: 0.1u, Capacitor_SMD:C_0603_1608Metric, F.Cu at (231.7, 53.0)
- added C146: 0.1u, Capacitor_SMD:C_0603_1608Metric, F.Cu at (236.6, 38.7)
- added C147: 10p, Capacitor_SMD:C_0603_1608Metric, F.Cu at (234.0, 56.3)
- added C148: 0.1u, Capacitor_SMD:C_0603_1608Metric, F.Cu at (234.0, 57.9)
- added C149: 0.1u, Capacitor_SMD:C_0603_1608Metric, F.Cu at (244.9, 59.0)
- added C15: 470u, Capacitor_SMD:C_0603_1608Metric, F.Cu at (85.8, 79.2)
- added C150: 0.1u, Capacitor_SMD:C_0603_1608Metric, F.Cu at (237.3, 63.0)
- added C151: 0.1u, Capacitor_SMD:C_0603_1608Metric, F.Cu at (206.3, 45.8)
- added C152: 0.1u, Capacitor_SMD:C_0603_1608Metric, F.Cu at (195.1, 47.2)
- added C153: 0.1u, Capacitor_SMD:C_0603_1608Metric, F.Cu at (105.8, 119.4)
- added C154: 0.1u, Capacitor_SMD:C_0603_1608Metric, F.Cu at (105.8, 120.9)
- added C155: 0.1u, Capacitor_SMD:C_0603_1608Metric, F.Cu at (84.6, 131.4)
- added C156: 0.1u, Capacitor_SMD:C_0603_1608Metric, F.Cu at (83.1, 131.4)
- added C157: 0.1u, Capacitor_SMD:C_0603_1608Metric, F.Cu at (86.5, 110.2)
- added C158: 0.1u, Capacitor_SMD:C_0603_1608Metric, F.Cu at (97.0, 111.7)
- added C159: 0.1u, Capacitor_SMD:C_0603_1608Metric, F.Cu at (88.0, 110.2)
- added C16: 10u, Capacitor_SMD:C_0603_1608Metric, F.Cu at (97.7, 63.9)
- added C160: 0.1u, Capacitor_SMD:C_0603_1608Metric, F.Cu at (98.8, 125.9)
- added C161: 0.1u, Capacitor_SMD:C_0603_1608Metric, F.Cu at (98.8, 128.2)
- added C162: 0.1u, Capacitor_SMD:C_0603_1608Metric, F.Cu at (97.0, 113.2)
- added C163: 0.1u, Capacitor_SMD:C_0603_1608Metric, F.Cu at (77.8, 113.7)
- added C164: 0.1u, Capacitor_SMD:C_0603_1608Metric, F.Cu at (81.2, 112.4)
- added C165: 0.1u, Capacitor_SMD:C_0603_1608Metric, F.Cu at (73.7, 120.7)
- added C166: 0.1u, Capacitor_SMD:C_0603_1608Metric, F.Cu at (73.7, 119.2)
- added C167: 0.1u, Capacitor_SMD:C_0603_1608Metric, F.Cu at (91.3, 135.5)
- added C168: 0.1u, Capacitor_SMD:C_0603_1608Metric, F.Cu at (89.5, 135.5)
- added C169: 0.1u, Capacitor_SMD:C_0603_1608Metric, F.Cu at (77.8, 115.2)
- added C17: 10u, Capacitor_SMD:C_0603_1608Metric, F.Cu at (97.7, 72.7)
- added C170: 0.1u, Capacitor_SMD:C_0603_1608Metric, F.Cu at (225.5, 127.3)
- added C171: 0.1u, Capacitor_SMD:C_0603_1608Metric, F.Cu at (238.7, 127.3)
- added C172: 0.1u, Capacitor_SMD:C_0603_1608Metric, F.Cu at (95.4, 114.8)
- added C173: 0.1u, Capacitor_SMD:C_0603_1608Metric, F.Cu at (100.4, 118.3)
- added C174: 0.1u, Capacitor_SMD:C_0603_1608Metric, F.Cu at (94.4, 124.3)
- added C175: 0.1u, Capacitor_SMD:C_0603_1608Metric, F.Cu at (96.6, 122.0)
- added C176: 0.1u, Capacitor_SMD:C_0603_1608Metric, F.Cu at (95.1, 122.0)
- added C177: 0.1u, Capacitor_SMD:C_0603_1608Metric, F.Cu at (92.2, 126.9)
- added C178: 0.1u, Capacitor_SMD:C_0603_1608Metric, F.Cu at (90.7, 125.8)
- added C179: 0.1u, Capacitor_SMD:C_0603_1608Metric, F.Cu at (88.5, 125.8)
- added C18: 2.2u, Capacitor_SMD:C_0603_1608Metric, F.Cu at (89.8, 79.2)
- added C180: 0.1u, Capacitor_SMD:C_0603_1608Metric, F.Cu at (87.0, 125.8)
- added C181: 0.1u, Capacitor_SMD:C_0603_1608Metric, F.Cu at (83.5, 124.4)
- added C182: 0.1u, Capacitor_SMD:C_0603_1608Metric, F.Cu at (85.8, 113.2)
- added C183: 0.1u, Capacitor_SMD:C_0603_1608Metric, F.Cu at (89.5, 111.9)
- added C184: 0.1u, Capacitor_SMD:C_0603_1608Metric, F.Cu at (91.0, 111.9)
- added C185: 0.1u, Capacitor_SMD:C_0603_1608Metric, F.Cu at (92.5, 111.9)
- added C186: 0.1u, Capacitor_SMD:C_0603_1608Metric, F.Cu at (82.5, 123.0)
- added C187: 0.1u, Capacitor_SMD:C_0603_1608Metric, F.Cu at (82.5, 121.4)
- added C188: 0.1u, Capacitor_SMD:C_0603_1608Metric, F.Cu at (83.4, 118.7)
- added C189: 0.1u, Capacitor_SMD:C_0603_1608Metric, F.Cu at (95.6, 116.6)
- added C19: 10u, Capacitor_SMD:C_0603_1608Metric, F.Cu at (98.0, 54.4)
- added C2: 27p, Capacitor_SMD:C_0603_1608Metric, F.Cu at (87.5, 97.4)
- added C20: 10u, Capacitor_SMD:C_0603_1608Metric, F.Cu at (112.7, 68.9)
- added C21: 10u, Capacitor_SMD:C_0603_1608Metric, F.Cu at (112.7, 59.9)
- added C22: 10u, Capacitor_SMD:C_0603_1608Metric, F.Cu at (78.1, 76.2)
- added C23: 10u, Capacitor_SMD:C_0603_1608Metric, F.Cu at (112.7, 50.4)
- added C24: 0.1u, Capacitor_SMD:C_0603_1608Metric, F.Cu at (124.1, 139.5)
- added C25: 0.1u, Capacitor_SMD:C_0603_1608Metric, F.Cu at (140.1, 137.9)
- added C26: 0.1u, Capacitor_SMD:C_0603_1608Metric, F.Cu at (140.1, 139.7)
- added C27: 1.5p, Capacitor_SMD:C_0603_1608Metric, F.Cu at (149.3, 146.2)
- added C28: 1.5p, Capacitor_SMD:C_0603_1608Metric, F.Cu at (149.3, 149.2)
- added C29: 1.5p, Capacitor_SMD:C_0603_1608Metric, F.Cu at (149.3, 130.9)
- added C3: 0.1u, Capacitor_SMD:C_0603_1608Metric, F.Cu at (85.4, 94.0)
- added C30: 1.5p, Capacitor_SMD:C_0603_1608Metric, F.Cu at (149.3, 127.8)
- added C31: 0.1u, Capacitor_SMD:C_0603_1608Metric, F.Cu at (125.8, 136.2)
- added C32: 0.1u, Capacitor_SMD:C_0603_1608Metric, F.Cu at (136.6, 138.8)
- added C33: 0.1u, Capacitor_SMD:C_0603_1608Metric, F.Cu at (127.2, 140.6)
- added C34: 0.1u, Capacitor_SMD:C_0603_1608Metric, F.Cu at (132.3, 132.8)
- added C35: 0.1u, Capacitor_SMD:C_0603_1608Metric, F.Cu at (132.3, 144.1)
- added C36: 1.5p, Capacitor_SMD:C_0603_1608Metric, F.Cu at (149.3, 140.1)
- added C37: 1.5p, Capacitor_SMD:C_0603_1608Metric, F.Cu at (149.3, 143.1)
- added C38: 1.5p, Capacitor_SMD:C_0603_1608Metric, F.Cu at (149.4, 133.9)
- added C39: 1.5p, Capacitor_SMD:C_0603_1608Metric, F.Cu at (149.4, 137.0)
- added C4: 1u, Capacitor_SMD:C_0603_1608Metric, F.Cu at (68.0, 96.2)
- added C40: 0.1u, Capacitor_SMD:C_0603_1608Metric, F.Cu at (164.1, 135.1)
- added C41: 0.1u, Capacitor_SMD:C_0603_1608Metric, F.Cu at (167.3, 131.1)
- added C42: 0.1u, Capacitor_SMD:C_0603_1608Metric, F.Cu at (163.7, 151.2)
- added C43: 0.1u, Capacitor_SMD:C_0603_1608Metric, F.Cu at (169.0, 147.1)
- added C44: 0.1u, Capacitor_SMD:C_0603_1608Metric, F.Cu at (162.2, 126.6)
- added C45: 0.1u, Capacitor_SMD:C_0603_1608Metric, F.Cu at (157.2, 130.5)
- added C46: 0.1u, Capacitor_SMD:C_0603_1608Metric, F.Cu at (161.7, 141.8)
- added C47: 0.1u, Capacitor_SMD:C_0603_1608Metric, F.Cu at (156.9, 146.1)
- added C48: 1u, Capacitor_SMD:C_0603_1608Metric, F.Cu at (177.1, 148.5)
- added C49: 1u, Capacitor_SMD:C_0603_1608Metric, F.Cu at (177.1, 145.4)
- added C5: 0.1u, Capacitor_SMD:C_0603_1608Metric, F.Cu at (66.1, 90.7)
- added C50: 1u, Capacitor_SMD:C_0603_1608Metric, F.Cu at (177.0, 132.7)
- added C51: 1u, Capacitor_SMD:C_0603_1608Metric, F.Cu at (177.0, 129.6)
- added C52: 0.1u, Capacitor_SMD:C_0603_1608Metric, F.Cu at (124.1, 108.3)
- added C53: 0.1u, Capacitor_SMD:C_0603_1608Metric, F.Cu at (140.1, 106.7)
- added C54: 0.1u, Capacitor_SMD:C_0603_1608Metric, F.Cu at (140.1, 108.5)
- added C55: 1.5p, Capacitor_SMD:C_0603_1608Metric, F.Cu at (149.3, 115.0)
- added C56: 1.5p, Capacitor_SMD:C_0603_1608Metric, F.Cu at (149.3, 118.0)
- added C57: 1.5p, Capacitor_SMD:C_0603_1608Metric, F.Cu at (149.3, 99.7)
- added C58: 1.5p, Capacitor_SMD:C_0603_1608Metric, F.Cu at (149.3, 96.6)
- added C59: 0.1u, Capacitor_SMD:C_0603_1608Metric, F.Cu at (125.8, 105.0)
- added C6: 0.1u, Capacitor_SMD:C_0603_1608Metric, F.Cu at (75.6, 89.2)
- added C60: 0.1u, Capacitor_SMD:C_0603_1608Metric, F.Cu at (136.6, 107.6)
- added C61: 0.1u, Capacitor_SMD:C_0603_1608Metric, F.Cu at (127.2, 109.4)
- added C62: 0.1u, Capacitor_SMD:C_0603_1608Metric, F.Cu at (132.3, 101.6)
- added C63: 0.1u, Capacitor_SMD:C_0603_1608Metric, F.Cu at (132.3, 112.9)
- added C64: 1.5p, Capacitor_SMD:C_0603_1608Metric, F.Cu at (149.4, 108.8)
- added C65: 1.5p, Capacitor_SMD:C_0603_1608Metric, F.Cu at (149.3, 111.9)
- added C66: 1.5p, Capacitor_SMD:C_0603_1608Metric, F.Cu at (149.4, 102.7)
- added C67: 1.5p, Capacitor_SMD:C_0603_1608Metric, F.Cu at (149.4, 105.8)
- added C68: 0.1u, Capacitor_SMD:C_0603_1608Metric, F.Cu at (164.1, 103.8)
- added C69: 0.1u, Capacitor_SMD:C_0603_1608Metric, F.Cu at (167.3, 99.9)
- added C7: 1u, Capacitor_SMD:C_0603_1608Metric, F.Cu at (68.6, 91.5)
- added C70: 0.1u, Capacitor_SMD:C_0603_1608Metric, F.Cu at (163.7, 120.0)
- added C71: 0.1u, Capacitor_SMD:C_0603_1608Metric, F.Cu at (169.0, 115.9)
- added C72: 0.1u, Capacitor_SMD:C_0603_1608Metric, F.Cu at (162.2, 95.4)
- added C73: 0.1u, Capacitor_SMD:C_0603_1608Metric, F.Cu at (157.2, 99.3)
- added C74: 0.1u, Capacitor_SMD:C_0603_1608Metric, F.Cu at (161.7, 110.6)
- added C75: 0.1u, Capacitor_SMD:C_0603_1608Metric, F.Cu at (156.9, 114.9)
- added C76: 1u, Capacitor_SMD:C_0603_1608Metric, F.Cu at (177.1, 117.3)
- added C77: 1u, Capacitor_SMD:C_0603_1608Metric, F.Cu at (177.1, 114.2)
- added C78: 1u, Capacitor_SMD:C_0603_1608Metric, F.Cu at (177.0, 101.5)
- added C79: 1u, Capacitor_SMD:C_0603_1608Metric, F.Cu at (177.0, 98.4)
- added C8: 0.1u, Capacitor_SMD:C_0603_1608Metric, F.Cu at (70.9, 89.8)
- added C80: 0.1u, Capacitor_SMD:C_0603_1608Metric, F.Cu at (124.1, 77.1)
- added C81: 0.1u, Capacitor_SMD:C_0603_1608Metric, F.Cu at (140.1, 75.5)
- added C82: 0.1u, Capacitor_SMD:C_0603_1608Metric, F.Cu at (140.1, 77.3)
- added C83: 1.5p, Capacitor_SMD:C_0603_1608Metric, F.Cu at (149.3, 83.7)
- added C84: 1.5p, Capacitor_SMD:C_0603_1608Metric, F.Cu at (149.3, 86.8)
- added C85: 1.5p, Capacitor_SMD:C_0603_1608Metric, F.Cu at (149.3, 68.5)
- added C86: 1.5p, Capacitor_SMD:C_0603_1608Metric, F.Cu at (149.3, 65.4)
- added C87: 0.1u, Capacitor_SMD:C_0603_1608Metric, F.Cu at (125.8, 73.8)
- added C88: 0.1u, Capacitor_SMD:C_0603_1608Metric, F.Cu at (136.6, 76.4)
- added C89: 0.1u, Capacitor_SMD:C_0603_1608Metric, F.Cu at (127.2, 78.2)
- added C9: 0.1u, Capacitor_SMD:C_0603_1608Metric, F.Cu at (82.6, 95.5)
- added C90: 0.1u, Capacitor_SMD:C_0603_1608Metric, F.Cu at (132.3, 70.4)
- added C91: 0.1u, Capacitor_SMD:C_0603_1608Metric, F.Cu at (132.3, 81.7)
- added C92: 1.5p, Capacitor_SMD:C_0603_1608Metric, F.Cu at (149.3, 77.6)
- added C93: 1.5p, Capacitor_SMD:C_0603_1608Metric, F.Cu at (149.3, 80.7)
- added C94: 1.5p, Capacitor_SMD:C_0603_1608Metric, F.Cu at (149.4, 71.5)
- added C95: 1.5p, Capacitor_SMD:C_0603_1608Metric, F.Cu at (149.4, 74.6)
- added C96: 0.1u, Capacitor_SMD:C_0603_1608Metric, F.Cu at (164.1, 72.6)
- added C97: 0.1u, Capacitor_SMD:C_0603_1608Metric, F.Cu at (167.3, 68.7)
- added C98: 0.1u, Capacitor_SMD:C_0603_1608Metric, F.Cu at (163.7, 88.8)
- added C99: 0.1u, Capacitor_SMD:C_0603_1608Metric, F.Cu at (169.0, 84.7)
- added D1: PMEG3020CEP, Diode_SMD:D_0603_1608Metric, F.Cu at (65.2, 48.3)
- added F1: F0603E1R25FSTR, Fuse:Fuse_0603_1608Metric, F.Cu at (68.3, 48.3)
- added J1: SWD_JP, Connector_PinSocket_1.00mm:PinSocket_1x02_P1.00mm_Vertical, F.Cu at (86.1, 87.8)
- added J2: 629105150521, Connector_USB:USB_Micro-B_Wuerth_629105150521, F.Cu at (58.4, 69.0)
- added J3: Conn_02x16, Connector_PinHeader_2.54mm:PinHeader_2x16_P2.54mm_Vertical, B.Cu at (201.1, 73.0)
- added J4: Barrel_Jack, Connector_BarrelJack:BarrelJack_Horizontal, F.Cu at (68.3, 54.8)
- added J5: CLK4_DIAG, Connector_PinHeader_2.54mm:PinHeader_1x02_P2.54mm_Vertical, F.Cu at (89.0, 142.2)
- added L1: 18u, Inductor_SMD:L_0603_1608Metric, F.Cu at (89.1, 75.4)
- added PS1: IA0515D, Converter_DCDC:Converter_DCDC_XP_POWER-IAxxxxD_THT, F.Cu at (88.2, 63.3)
- added R1: 27.4, Resistor_SMD:R_0603_1608Metric, F.Cu at (61.8, 89.8)
- added R10: 499, Resistor_SMD:R_0603_1608Metric, F.Cu at (147.8, 146.2)
- added R100: 1k, Resistor_SMD:R_0603_1608Metric, F.Cu at (174.0, 38.4)
- added R101: 1k, Resistor_SMD:R_0603_1608Metric, F.Cu at (174.0, 35.3)
- added R102: 49.9, Resistor_SMD:R_0603_1608Metric, F.Cu at (175.6, 54.1)
- added R103: 49.9, Resistor_SMD:R_0603_1608Metric, F.Cu at (175.6, 51.0)
- added R104: 49.9, Resistor_SMD:R_0603_1608Metric, F.Cu at (175.6, 38.4)
- added R105: 49.9, Resistor_SMD:R_0603_1608Metric, F.Cu at (175.6, 35.3)
- added R106: 1M, Resistor_SMD:R_0603_1608Metric, F.Cu at (220.1, 59.2)
- added R107: 1M, Resistor_SMD:R_0603_1608Metric, F.Cu at (228.1, 59.2)
- added R109: 1M, Resistor_SMD:R_0603_1608Metric, F.Cu at (234.8, 54.0)
- added R11: 499, Resistor_SMD:R_0603_1608Metric, F.Cu at (147.8, 149.2)
- added R110: 10k, Resistor_SMD:R_0603_1608Metric, F.Cu at (234.8, 60.1)
- added R111: 100k, Resistor_SMD:R_0603_1608Metric, F.Cu at (237.3, 59.2)
- added R113: 1k, Resistor_SMD:R_0603_1608Metric, F.Cu at (192.8, 40.7)
- added R114: 1k, Resistor_SMD:R_0603_1608Metric, F.Cu at (189.7, 47.1)
- added R115: 1k, Resistor_SMD:R_0603_1608Metric, F.Cu at (192.8, 42.3)
- added R116: 500, Resistor_SMD:R_0603_1608Metric, F.Cu at (192.7, 51.9)
- added R117: 500, Resistor_SMD:R_0603_1608Metric, F.Cu at (206.3, 49.6)
- added R119: 240, Resistor_SMD:R_0603_1608Metric, F.Cu at (105.3, 123.4)
- added R12: 499, Resistor_SMD:R_0603_1608Metric, F.Cu at (147.8, 130.9)
- added R120: 240, Resistor_SMD:R_0603_1608Metric, F.Cu at (82.3, 129.2)
- added R121: 240, Resistor_SMD:R_0603_1608Metric, F.Cu at (105.3, 116.9)
- added R122: 240, Resistor_SMD:R_0603_1608Metric, F.Cu at (85.3, 129.2)
- added R123: 100, Resistor_SMD:R_0603_1608Metric, F.Cu at (103.6, 120.2)
- added R124: 100, Resistor_SMD:R_0603_1608Metric, F.Cu at (83.8, 127.7)
- added R125: 100, Resistor_SMD:R_0603_1608Metric, F.Cu at (96.5, 127.0)
- added R126: 240, Resistor_SMD:R_0603_1608Metric, F.Cu at (76.0, 118.4)
- added R127: 240, Resistor_SMD:R_0603_1608Metric, F.Cu at (76.0, 121.5)
- added R128: 4.12k, Resistor_SMD:R_0603_1608Metric, F.Cu at (98.8, 115.5)
- added R129: 100, Resistor_SMD:R_0603_1608Metric, F.Cu at (77.5, 119.9)
- added R13: 499, Resistor_SMD:R_0603_1608Metric, F.Cu at (147.8, 127.8)
- added R130: 50, Resistor_SMD:R_0603_1608Metric, F.Cu at (81.2, 110.9)
- added R131: 100, Resistor_SMD:R_0603_1608Metric, F.Cu at (90.3, 133.0)
- added R14: 499, Resistor_SMD:R_0603_1608Metric, F.Cu at (146.2, 140.1)
- added R15: 499, Resistor_SMD:R_0603_1608Metric, F.Cu at (146.2, 143.1)
- added R16: 499, Resistor_SMD:R_0603_1608Metric, F.Cu at (146.3, 133.9)
- added R17: 499, Resistor_SMD:R_0603_1608Metric, F.Cu at (146.3, 137.0)
- added R18: 499, Resistor_SMD:R_0603_1608Metric, F.Cu at (147.8, 140.1)
- added R19: 499, Resistor_SMD:R_0603_1608Metric, F.Cu at (147.8, 143.1)
- added R2: 27.4, Resistor_SMD:R_0603_1608Metric, F.Cu at (63.3, 89.9)
- added R20: 499, Resistor_SMD:R_0603_1608Metric, F.Cu at (147.8, 133.9)
- added R21: 499, Resistor_SMD:R_0603_1608Metric, F.Cu at (147.8, 137.0)
- added R22: 8.06K, Resistor_SMD:R_0603_1608Metric, F.Cu at (128.4, 144.1)
- added R23: 1k, Resistor_SMD:R_0603_1608Metric, F.Cu at (174.0, 148.5)
- added R24: 1k, Resistor_SMD:R_0603_1608Metric, F.Cu at (174.0, 145.4)
- added R25: 1k, Resistor_SMD:R_0603_1608Metric, F.Cu at (173.9, 132.7)
- added R26: 1k, Resistor_SMD:R_0603_1608Metric, F.Cu at (173.9, 129.6)
- added R27: 49.9, Resistor_SMD:R_0603_1608Metric, F.Cu at (175.5, 148.5)
- added R28: 49.9, Resistor_SMD:R_0603_1608Metric, F.Cu at (175.5, 145.4)
- added R29: 49.9, Resistor_SMD:R_0603_1608Metric, F.Cu at (175.5, 132.7)
- added R3: 1k, Resistor_SMD:R_0603_1608Metric, F.Cu at (88.5, 94.4)
- added R30: 49.9, Resistor_SMD:R_0603_1608Metric, F.Cu at (175.5, 129.6)
- added R31: 499, Resistor_SMD:R_0603_1608Metric, F.Cu at (146.2, 115.0)
- added R32: 499, Resistor_SMD:R_0603_1608Metric, F.Cu at (146.2, 118.0)
- added R33: 499, Resistor_SMD:R_0603_1608Metric, F.Cu at (146.2, 99.7)
- added R34: 499, Resistor_SMD:R_0603_1608Metric, F.Cu at (146.2, 96.6)
- added R35: 499, Resistor_SMD:R_0603_1608Metric, F.Cu at (147.8, 115.0)
- added R36: 499, Resistor_SMD:R_0603_1608Metric, F.Cu at (147.8, 118.0)
- added R37: 499, Resistor_SMD:R_0603_1608Metric, F.Cu at (147.8, 99.7)
- added R38: 499, Resistor_SMD:R_0603_1608Metric, F.Cu at (147.8, 96.6)
- added R39: 499, Resistor_SMD:R_0603_1608Metric, F.Cu at (146.3, 108.8)
- added R4: 1k, Resistor_SMD:R_0603_1608Metric, F.Cu at (60.8, 108.2)
- added R40: 499, Resistor_SMD:R_0603_1608Metric, F.Cu at (146.2, 111.9)
- added R41: 499, Resistor_SMD:R_0603_1608Metric, F.Cu at (146.3, 102.7)
- added R42: 499, Resistor_SMD:R_0603_1608Metric, F.Cu at (146.3, 105.8)
- added R43: 499, Resistor_SMD:R_0603_1608Metric, F.Cu at (147.8, 108.8)
- added R44: 499, Resistor_SMD:R_0603_1608Metric, F.Cu at (147.8, 111.9)
- added R45: 499, Resistor_SMD:R_0603_1608Metric, F.Cu at (147.8, 102.7)
- added R46: 499, Resistor_SMD:R_0603_1608Metric, F.Cu at (147.8, 105.8)
- added R47: 8.06K, Resistor_SMD:R_0603_1608Metric, F.Cu at (128.4, 112.9)
- added R48: 1k, Resistor_SMD:R_0603_1608Metric, F.Cu at (174.0, 117.3)
- added R49: 1k, Resistor_SMD:R_0603_1608Metric, F.Cu at (174.0, 114.2)
- added R5: 4.7k, Resistor_SMD:R_0603_1608Metric, F.Cu at (60.8, 117.2)
- added R50: 1k, Resistor_SMD:R_0603_1608Metric, F.Cu at (173.9, 101.5)
- added R51: 1k, Resistor_SMD:R_0603_1608Metric, F.Cu at (173.9, 98.4)
- added R52: 49.9, Resistor_SMD:R_0603_1608Metric, F.Cu at (175.5, 117.3)
- added R53: 49.9, Resistor_SMD:R_0603_1608Metric, F.Cu at (175.5, 114.2)
- added R54: 49.9, Resistor_SMD:R_0603_1608Metric, F.Cu at (175.5, 101.5)
- added R55: 49.9, Resistor_SMD:R_0603_1608Metric, F.Cu at (175.5, 98.4)
- added R56: 499, Resistor_SMD:R_0603_1608Metric, F.Cu at (146.2, 83.7)
- added R57: 499, Resistor_SMD:R_0603_1608Metric, F.Cu at (146.2, 86.8)
- added R58: 499, Resistor_SMD:R_0603_1608Metric, F.Cu at (146.2, 68.5)
- added R59: 499, Resistor_SMD:R_0603_1608Metric, F.Cu at (146.2, 65.4)
- added R6: 499, Resistor_SMD:R_0603_1608Metric, F.Cu at (146.2, 146.2)
- added R60: 499, Resistor_SMD:R_0603_1608Metric, F.Cu at (147.8, 83.7)
- added R61: 499, Resistor_SMD:R_0603_1608Metric, F.Cu at (147.8, 86.8)
- added R62: 499, Resistor_SMD:R_0603_1608Metric, F.Cu at (147.8, 68.5)
- added R63: 499, Resistor_SMD:R_0603_1608Metric, F.Cu at (147.8, 65.4)
- added R64: 499, Resistor_SMD:R_0603_1608Metric, F.Cu at (146.2, 77.6)
- added R65: 499, Resistor_SMD:R_0603_1608Metric, F.Cu at (146.2, 80.7)
- added R66: 499, Resistor_SMD:R_0603_1608Metric, F.Cu at (146.3, 71.5)
- added R67: 499, Resistor_SMD:R_0603_1608Metric, F.Cu at (146.3, 74.6)
- added R68: 499, Resistor_SMD:R_0603_1608Metric, F.Cu at (147.8, 77.6)
- added R69: 499, Resistor_SMD:R_0603_1608Metric, F.Cu at (147.8, 80.7)
- added R7: 499, Resistor_SMD:R_0603_1608Metric, F.Cu at (146.2, 149.2)
- added R70: 499, Resistor_SMD:R_0603_1608Metric, F.Cu at (147.8, 71.5)
- added R71: 499, Resistor_SMD:R_0603_1608Metric, F.Cu at (147.8, 74.6)
- added R72: 8.06K, Resistor_SMD:R_0603_1608Metric, F.Cu at (128.4, 81.7)
- added R73: 1k, Resistor_SMD:R_0603_1608Metric, F.Cu at (174.0, 86.1)
- added R74: 1k, Resistor_SMD:R_0603_1608Metric, F.Cu at (174.0, 82.9)
- added R75: 1k, Resistor_SMD:R_0603_1608Metric, F.Cu at (173.9, 70.3)
- added R76: 1k, Resistor_SMD:R_0603_1608Metric, F.Cu at (173.9, 67.2)
- added R77: 49.9, Resistor_SMD:R_0603_1608Metric, F.Cu at (175.5, 86.1)
- added R78: 49.9, Resistor_SMD:R_0603_1608Metric, F.Cu at (175.5, 82.9)
- added R79: 49.9, Resistor_SMD:R_0603_1608Metric, F.Cu at (175.5, 70.3)
- added R8: 499, Resistor_SMD:R_0603_1608Metric, F.Cu at (146.2, 130.9)
- added R80: 49.9, Resistor_SMD:R_0603_1608Metric, F.Cu at (175.5, 67.2)
- added R81: 499, Resistor_SMD:R_0603_1608Metric, F.Cu at (146.4, 51.8)
- added R82: 499, Resistor_SMD:R_0603_1608Metric, F.Cu at (146.4, 54.9)
- added R83: 499, Resistor_SMD:R_0603_1608Metric, F.Cu at (146.4, 36.5)
- added R84: 499, Resistor_SMD:R_0603_1608Metric, F.Cu at (146.4, 33.5)
- added R85: 499, Resistor_SMD:R_0603_1608Metric, F.Cu at (147.9, 51.8)
- added R86: 499, Resistor_SMD:R_0603_1608Metric, F.Cu at (147.9, 54.9)
- added R87: 499, Resistor_SMD:R_0603_1608Metric, F.Cu at (147.9, 36.5)
- added R88: 499, Resistor_SMD:R_0603_1608Metric, F.Cu at (147.9, 33.5)
- added R89: 499, Resistor_SMD:R_0603_1608Metric, F.Cu at (146.4, 45.7)
- added R9: 499, Resistor_SMD:R_0603_1608Metric, F.Cu at (146.2, 127.8)
- added R90: 499, Resistor_SMD:R_0603_1608Metric, F.Cu at (146.4, 48.7)
- added R91: 499, Resistor_SMD:R_0603_1608Metric, F.Cu at (146.4, 39.6)
- added R92: 499, Resistor_SMD:R_0603_1608Metric, F.Cu at (146.4, 42.6)
- added R93: 499, Resistor_SMD:R_0603_1608Metric, F.Cu at (147.9, 45.7)
- added R94: 499, Resistor_SMD:R_0603_1608Metric, F.Cu at (147.9, 48.7)
- added R95: 499, Resistor_SMD:R_0603_1608Metric, F.Cu at (147.9, 39.6)
- added R96: 499, Resistor_SMD:R_0603_1608Metric, F.Cu at (147.9, 42.6)
- added R97: 8.06K, Resistor_SMD:R_0603_1608Metric, F.Cu at (128.6, 49.8)
- added R98: 1k, Resistor_SMD:R_0603_1608Metric, F.Cu at (174.1, 54.1)
- added R99: 1k, Resistor_SMD:R_0603_1608Metric, F.Cu at (174.1, 51.0)
- added REF**: MountingHole_3.2mm_M3_DIN965_Pad, MountingHole:MountingHole_3.2mm_M3_DIN965_Pad, F.Cu at (246.9, 149.5)
- added REF**: MountingHole_3.2mm_M3_DIN965_Pad, MountingHole:MountingHole_3.2mm_M3_DIN965_Pad, F.Cu at (62.1, 149.5)
- added REF**: MountingHole_3.2mm_M3_DIN965_Pad, MountingHole:MountingHole_3.2mm_M3_DIN965_Pad, F.Cu at (247.1, 34.5)
- added REF**: MountingHole_3.2mm_M3_DIN965_Pad, MountingHole:MountingHole_3.2mm_M3_DIN965_Pad, F.Cu at (62.1, 34.5)
- added RV1: M64W202KB40, M64W103KB40:POT_2023-08-01_VIS, F.Cu at (226.1, 34.2)
- added RV2: M64W202KB40, M64W103KB40:POT_2023-08-01_VIS, F.Cu at (195.4, 33.8)
- added RV3: M64W103KB40, M64W103KB40:POT_2023-08-01_VIS, F.Cu at (206.9, 55.9)
- added SW1: SKRKAHE020, Button_Switch_SMD:SW_Push_SPST_NO_Alps_SKRK, F.Cu at (62.8, 111.9)
- added SW2: SKRKAHE020, Button_Switch_SMD:SW_Push_SPST_NO_Alps_SKRK, F.Cu at (62.8, 121.2)
- added SW3: ANT11SF1CQE, ANT11SF1CQE:ANT11SF1CQE, F.Cu at (65.3, 42.5)
- added SW4: SW_SPDT_321, Button_Switch_THT:SW_E-Switch_EG1271_SPDT, F.Cu at (186.9, 39.9)
- added U1: RP2040, Package_DFN_QFN:QFN-56-1EP_7x7mm_P0.4mm_EP3.2x3.2mm, F.Cu at (75.1, 96.0)
- added U10: ADA4817-2ACPZ-R7, ADA4817-2ACPZ-R7:CP_16_4_ADI, F.Cu at (162.7, 115.6)
- added U11: ADA4817-2ACPZ-R7, ADA4817-2ACPZ-R7:CP_16_4_ADI, F.Cu at (163.2, 99.6)
- added U12: AD9106BCP, Package_CSP:LFCSP-32-1EP_5x5mm_P0.5mm_EP3.6x3.6mm, F.Cu at (132.1, 76.2)
- added U13: ADA4817-2ACPZ-R7, ADA4817-2ACPZ-R7:CP_16_4_ADI, F.Cu at (162.7, 84.4)
- added U14: ADA4817-2ACPZ-R7, ADA4817-2ACPZ-R7:CP_16_4_ADI, F.Cu at (163.2, 68.4)
- added U15: AD9106BCP, Package_CSP:LFCSP-32-1EP_5x5mm_P0.5mm_EP3.6x3.6mm, F.Cu at (132.2, 44.3)
- added U16: ADA4817-2ACPZ-R7, ADA4817-2ACPZ-R7:CP_16_4_ADI, F.Cu at (162.8, 52.5)
- added U17: ADA4817-2ACPZ-R7, ADA4817-2ACPZ-R7:CP_16_4_ADI, F.Cu at (163.3, 36.4)
- added U18: AD7680ARJZ-REEL7, AD7680ARJZ:RJ_6_ADI, F.Cu at (246.1, 66.6)
- added U19: TL071, Package_SO:TSSOP-8_3x3mm_P0.65mm, F.Cu at (217.4, 55.3)
- added U2: W25Q128JVS, Package_SO:SOIC-8_5.23x5.23mm_P1.27mm, F.Cu at (63.0, 101.9)
- added U20: TL071, Package_SO:TSSOP-8_3x3mm_P0.65mm, F.Cu at (225.4, 55.3)
- added U21: INA849DR, INA849DR:D0008A-IPC_A, F.Cu at (222.1, 42.8)
- added U22: AD630ARZ, Package_SO:SOIC-20W_7.5x12.8mm_P1.27mm, F.Cu at (238.6, 46.0)
- added U23: TL071, Package_SO:TSSOP-8_3x3mm_P0.65mm, F.Cu at (241.1, 60.6)
- added U24: OPA4228UA, OPA4228UA:D14, F.Cu at (201.1, 46.4)
- added U25: AD9512BCPZ, AD9512BCPZ:CP_48_1_ADI, F.Cu at (89.7, 119.4)
- added U26: SN74HC595, Package_SO:SOIC-16W_5.3x10.2mm_P1.27mm, F.Cu at (220.3, 121.8)
- added U27: SN74HC595, Package_SO:SOIC-16W_5.3x10.2mm_P1.27mm, F.Cu at (233.5, 121.8)
- added U28: ADG1406BRUZ-REEL7, ADG1406BRUZ:RU_28_ADI, F.Cu at (209.7, 91.9)
- added U29: ADG1406BRUZ-REEL7, ADG1406BRUZ:RU_28_ADI, F.Cu at (221.3, 91.9)
- added U3: NCP1117-3.3_SOT223, Package_TO_SOT_SMD:SOT-223-3_TabPin2, F.Cu at (104.9, 59.9)
- added U30: ADG1406BRUZ-REEL7, ADG1406BRUZ:RU_28_ADI, F.Cu at (233.0, 91.9)
- added U31: ADG1406BRUZ-REEL7, ADG1406BRUZ:RU_28_ADI, F.Cu at (244.5, 91.9)
- added U4: NCP1117-3.3_SOT223, Package_TO_SOT_SMD:SOT-223-3_TabPin2, F.Cu at (104.9, 68.9)
- added U5: NCP1117-5.0_SOT223, Package_TO_SOT_SMD:SOT-223-3_TabPin2, F.Cu at (104.7, 50.4)
- added U6: AD9106BCP, Package_CSP:LFCSP-32-1EP_5x5mm_P0.5mm_EP3.6x3.6mm, F.Cu at (132.1, 138.6)
- added U7: ADA4817-2ACPZ-R7, ADA4817-2ACPZ-R7:CP_16_4_ADI, F.Cu at (162.7, 146.8)
- added U8: ADA4817-2ACPZ-R7, ADA4817-2ACPZ-R7:CP_16_4_ADI, F.Cu at (163.2, 130.8)
- added U9: AD9106BCP, Package_CSP:LFCSP-32-1EP_5x5mm_P0.5mm_EP3.6x3.6mm, F.Cu at (132.1, 107.4)
- added Y1: ABLS-12.000MHZ-B4-T, Crystal:Crystal_SMD_HC49-SD, F.Cu at (94.0, 98.7)
Routing:
- net VSS: track 0.00 -> 867.7 mm, vias 0 -> 28
- net VCC: track 0.00 -> 725.1 mm, vias 0 -> 28
- net /SPI0_RX: track 0.00 -> 478.4 mm, vias 0 -> 7
- net /SPI0_SCLK: track 0.00 -> 450.9 mm, vias 0 -> 8
- net GND: track 0.00 -> 411.3 mm, vias 0 -> 233
- net +3.3V: track 0.00 -> 400.5 mm, vias 0 -> 21
- net +3.3VA: track 0.00 -> 399.8 mm, vias 0 -> 16
- net /~{AMP_PD}: track 0.00 -> 319.3 mm, vias 0 -> 19
- net /~{RESET}: track 0.00 -> 270.2 mm, vias 0 -> 11
- net /MUX_EN: track 0.00 -> 268.9 mm, vias 0 -> 5
- net /~{AN_CS}: track 0.00 -> 255.1 mm, vias 0 -> 2
- net /SPI0_TX: track 0.00 -> 254.3 mm, vias 0 -> 7
- net /~{DDS_SYNC}: track 0.00 -> 191.7 mm, vias 0 -> 7
- net /SR_CLK: track 0.00 -> 191.3 mm, vias 0 -> 6
- net /~{SR_OE}: track 0.00 -> 189.1 mm, vias 0 -> 5
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- added copper zone on In2.Cu, net +3.3V
- added copper zone on In2.Cu, net +3.3VA
- added copper zone on In1.Cu, net GND
- added copper zone on In2.Cu, net VCC
- added copper zone on In2.Cu, net VSS
Other:
- board outline added: 200 x 130 mm
- board text added: "BOOT_SEL"
- board text added: "ENEL 500 Group OM4 Prototype 16CH-EIT v0.1"
- board text added: "HDR1"
- board text added: "HDR15"
- board text added: "RESET"

Commit message: Slight board updates - Added board PDFs and images
Parts:
- J4: footprint Connector_BarrelJack:BarrelJack_Horizontal -> Connector_BarrelJack:BarrelJack_GCT_DCJ200-10-A_Horizontal
- SW1: value SKRKAHE020 -> BOOT_SEL
- SW2: value SKRKAHE020 -> SW_Push
- turned J4 to -90 degrees
Connections:
- C117 pad 1: Net-(U15-CLKVDD) -> +3.3V
- C118 pad 2: Net-(U15-AVDD1) -> +3.3VA
- C33 pad 1: Net-(U6-CLKVDD) -> +3.3V
- C34 pad 2: Net-(U6-AVDD1) -> +3.3VA
- C61 pad 1: Net-(U9-CLKVDD) -> +3.3V
- C62 pad 2: Net-(U9-AVDD1) -> +3.3VA
- C89 pad 1: Net-(U12-CLKVDD) -> +3.3V
- C90 pad 2: Net-(U12-AVDD1) -> +3.3VA
- J4 pad 3: (no net) -> GND
- U12 pad 23: Net-(U12-CLKVDD) -> +3.3V
- U12 pad 29: Net-(U12-AVDD1) -> +3.3VA
- U15 pad 23: Net-(U15-CLKVDD) -> +3.3V
- U15 pad 29: Net-(U15-AVDD1) -> +3.3VA
- U6 pad 23: Net-(U6-CLKVDD) -> +3.3V
- U6 pad 29: Net-(U6-AVDD1) -> +3.3VA
- U9 pad 23: Net-(U9-CLKVDD) -> +3.3V
- U9 pad 29: Net-(U9-AVDD1) -> +3.3VA
Routing:
- net +3.3VA: track 399.8 -> 425.6 mm, vias 16 -> 20
- net +3.3V: track 400.5 -> 408.2 mm
- net GND: track 411.3 -> 408.6 mm
- net Net-(U9-CLKVDD): track 1.94 -> 0.00 mm
- net Net-(U15-CLKVDD): track 1.94 -> 0.00 mm
- net Net-(U6-CLKVDD): track 1.94 -> 0.00 mm
- net Net-(U12-CLKVDD): track 1.94 -> 0.00 mm

Commit message: Final KiCAD Files Submitted to JLC PCB
Parts:
- added D2: PMEG3020CEP, Diode_SMD:D_0603_1608Metric, F.Cu at (65.7, 67.8)
- C15: footprint Capacitor_SMD:C_0603_1608Metric -> Capacitor_THT:CP_Radial_D6.3mm_P2.50mm
- J2: footprint Connector_USB:USB_Micro-B_Wuerth_629105150521 -> Connector_USB:USB_Micro-B_Amphenol_10118193-0001LF_Horizontal
- U19, U20, U23: value TL071 -> TL071HD; footprint Package_SO:TSSOP-8_3x3mm_P0.65mm -> Package_SO:SOIC-8_3.9x4.9mm_P1.27mm
- moved J2 13.0 mm to (56.1, 81.8)
- moved R106 1.61 mm to (219.7, 60.8), turned to 90 degrees
- moved C140 1.25 mm to (220.9, 57.6)
- moved C142 1.08 mm to (229.1, 56.9)
- moved C141 1.00 mm to (223.6, 50.5)
- moved R111 0.92 mm to (236.4, 59.2)
- moved C149 0.85 mm to (245.7, 59.2)
- moved C139 0.84 mm to (215.7, 50.6)
- moved C136 0.83 mm to (218.1, 60.8)
- moved C150 0.82 mm to (236.6, 63.4)
- moved C137 0.66 mm to (226.1, 60.6)
- moved R107 0.66 mm to (228.4, 59.8)
- moved C15 0.32 mm to (85.6, 79.0)
Connections:
- J2 pad 1: unconnected-(J2-VBUS-Pad1) -> VBUS
- SW3 pad 3: unconnected-(SW3-Pad3) -> GND
Routing:
- net Net-(D2-K): track 36.5 -> 57.4 mm
- net VBUS: track 0.00 -> 16.2 mm
- net /USB_D-: track 24.6 -> 10.0 mm
- net /USB_D+: track 23.1 -> 9.20 mm
- net GND: track 408.6 -> 406.3 mm, vias 233 -> 232
- net VSS: track 867.7 -> 869.3 mm, vias 28 -> 29
- net /Analog/ADC_IN: track 11.6 -> 13.0 mm
- net Net-(U1-USB_DM): track 10.4 -> 11.6 mm
- net VCC: track 725.1 -> 726.4 mm
- net Net-(U1-USB_DP): track 11.4 -> 12.2 mm
- net /Analog/SENSE_IN_1: track 29.4 -> 28.8 mm
- net +3.3V: track 408.2 -> 408.3 mm, vias 21 -> 24
Other:
- board text added: "*"
