File: PCB_Design/picoAWG.kicad_sch (KiCad schematic)
At the start: 27 parts, among them J1 SWD_JP, J2 USB_B_Micro, J3 Conn_02x16, SW1 BOOT_SEL, SW2 SW_Push, U1 RP2040, U2 W25Q128JVS, Y1 ABLS-12.000MHZ-B4-T

Commit message: KiCAD file update, completed PCB
Parts:
- added SW4: SW_SPDT_321, Button_Switch_THT:SW_E-Switch_EG1271_SPDT, symbol Switch:SW_SPDT_321
- J2: value USB_B_Micro -> 629105150521
Connections:
- net HDR_15: now also SW4.3 (A)
- new net Analog/CARRIER_SIG: SW4.1 (C)
- new net DDS 4/OUT4: SW4.2 (B)
Other:
- note added: "Clock assignment was modified for ease of routing."

Commit message: Final KiCAD Files Submitted to JLC PCB
Parts:
- J2: footprint Connector_USB:USB_Micro-B_Wuerth_629105150521 -> Connector_USB:USB_Micro-B_Amphenol_10118193-0001LF_Horizontal
Connections:
- net VBUS: now reaches J2.1 (VBUS)
- no-connect marks 11 -> 10
Changed lines of the file:
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@@
   (no_connect (at 160.02 129.54))
   (no_connect (at 92.71 133.35))
-  (no_connect (at 160.02 119.38))
   (no_connect (at 92.71 130.81))
   (no_connect (at 92.71 77.47))
@@
   )
   (wire (pts (xy 33.782 72.39) (xy 41.91 72.39))
+    (stroke (width 0) (type default))
+  )
+  (wire (pts (xy 160.02 119.38) (xy 163.83 119.38))
     (stroke (width 0) (type default))
   )
@@
       (effects (font (size 1.27 1.27)))
     )
-    (property "Footprint" "Connector_USB:USB_Micro-B_Wuerth_629105150521" (at 156.21 125.73 0)
+    (property "Footprint" "Connector_USB:USB_Micro-B_Amphenol_10118193-0001LF_Horizontal" (at 156.21 125.73 0)
       (effects (font (size 1.27 1.27)) hide)
     )
@@
         )
       )
+    )
+  )
+  (symbol (lib_id "power:VBUS") (at 163.83 119.38 0) (unit 1)
+    (in_bom yes) (on_board yes) (dnp no) (fields_autoplaced)
+    (property "Reference" "#PWR0249" (at 163.83 123.19 0)
+      (effects (font (size 1.27 1.27)) hide)
+    )
+    (property "Value" "VBUS" (at 163.83 114.3 0)
+      (effects (font (size 1.27 1.27)))
+    )
+    (property "Footprint" "" (at 163.83 119.38 0)
+      (effects (font (size 1.27 1.27)) hide)
+    )
+    (property "Datasheet" "" (at 163.83 119.38 0)
+      (effects (font (size 1.27 1.27)) hide)
+    )
+    (pin "1")
+    (instances
+      (project "picoAWG"
+        (path "/98622ba7-93bb-40c5-bd9c-32780137208f"
+          (reference "#PWR0249") (unit 1)
+        )
+      )
